File: cad/winder/PCB/winder_pcb/re_winder_pcb.kicad_pcb (KiCad board)
At the start: 2 copper layers, 51 x 108 mm, 37 parts, among them J1 12V_IN, M3 MountingHole_3.2mm_M3

Commit message: パワー基盤の作成完了
Parts:
- moved FAN_D1 10.7 mm to (112.0, 60.9)
- moved FAN_FET1 3.97 mm to (112.1, 66.5), turned to -90 degrees
Connections:
- FAN_D1 pad 1: Net-(FAN_D1-K) -> +12V
- FAN_FET1 pad 2: Net-(FAN_D1-K) -> Net-(FAN1--)
Routing:
- net Net-(FAN_D1-K): track 11.0 -> 0.00 mm
- net Net-(FAN1--): track 20.2 -> 12.3 mm
- net +12V: track 60.7 -> 67.9 mm
- net GND: track 390.3 -> 385.5 mm
- net Net-(FAN_FET1-G): track 13.1 -> 14.6 mm
